File: arduino_shield.sch (KiCad schematic (older format))
At the start: 10 parts, among them P1 Power, P2 Analog, P3 Digital, P4 Digital, P5 CONN_01X01, P6 CONN_01X01, P7 CONN_01X01, P8 CONN_01X01, U1 MS560702BA03-50

Commit message: finished maybe?
Parts:
- removed MOD1: XBP9B-DMST-002, digikey-footprints:XBEE_PRO-20_THT, symbol dk_RF-Transceiver-Modules:XBP9B-DMST-002
- removed U1: MS560702BA03-50, digikey-footprints:SMD-8_5x3mm, symbol dk_Pressure-Sensors-Transducers:MS560702BA03-50
- added J1: GND Rail, Connector_PinHeader_2.54mm:PinHeader_1x08_P2.54mm_Vertical, symbol Connector:Conn_01x08_Male
- added J2: 5V Rail, Connector_PinHeader_2.54mm:PinHeader_1x08_P2.54mm_Vertical, symbol Connector:Conn_01x08_Male
- added J3: 3v3 Rail, Connector_PinHeader_2.54mm:PinHeader_1x08_P2.54mm_Vertical, symbol Connector:Conn_01x08_Male
- added U1: XMEGA_A1U_Xplained_Pro, One_Month_Footprints:XMEGA_XPLAINED_AU, symbol One_Month_Board_Symbols:XMEGA_A1U_Xplained_Pro
Connections:
- net +3V3: now also J3.1 (Pin_1), J3.2 (Pin_2), J3.3 (Pin_3), J3.4 (Pin_4), J3.5 (Pin_5), J3.6 (Pin_6), J3.7 (Pin_7), J3.8 (Pin_8), U1.A20 (VCC), U1.B20 (VCC), U1.C20 (VCC), U1.P4 (VCC_P3V3)
- net +5V: now also J2.1 (Pin_1), J2.2 (Pin_2), J2.3 (Pin_3), J2.4 (Pin_4), J2.5 (Pin_5), J2.6 (Pin_6), J2.7 (Pin_7), J2.8 (Pin_8), U1.P3 (VCC_P5V0)
- net GND: now also J1.1 (Pin_1), J1.2 (Pin_2), J1.3 (Pin_3), J1.4 (Pin_4), J1.5 (Pin_5), J1.6 (Pin_6), J1.7 (Pin_7), J1.8 (Pin_8), U1.A19 (GND), U1.A2 (GND), U1.B19 (GND), U1.B2 (GND), U1.C19 (GND), U1.C2 (GND), U1.P2 (GND)
- no-connect marks 5 -> 57

Commit message: added pdf for schematic
Parts:
- added U?: MPU-9250, QFN40P300X300X105-25N, symbol MPU-9250:MPU-9250
Changed lines of the file:
@@
 	0    1    1    0
 $EndComp
+$Comp
+L MPU-9250:MPU-9250 U?
+U 1 1 5D715A4C
+P 2750 2950
+F 0 "U?" H 2750 3915 50  0000 C CNN
+F 1 "MPU-9250" H 2750 3824 50  0000 C CNN
+F 2 "QFN40P300X300X105-25N" H 2750 2950 50  0001 L BNN
+F 3 "" H 2750 2950 50  0001 L BNN
+F 4 "TDK InvenSense" H 2750 2950 50  0001 L BNN "Field4"
+F 5 "SMD Gyroscope/Accelerometer/Magnetometer Sensor; 9-AXIS" H 2750 2950 50  0001 L BNN "Field5"
+F 6 "QFN-24 TDK InvenSense" H 2750 2950 50  0001 L BNN "Field6"
+F 7 "Unavailable" H 2750 2950 50  0001 L BNN "Field7"
+F 8 "MPU-9250" H 2750 2950 50  0001 L BNN "Field8"
+	1    2750 2950
+	1    0    0    -1
+$EndComp
 $EndSCHEMATC
